Commit message: tt

File: map/scout_mini_omni.urdf (robot description, URDF)
Before this commit: robot scout_mini_omni, 5 links, 4 joints
Links:
- link base_link: mass 10 -> 23
- link front_left_wheel: geometry collision cylinder length=0.05 radius=0.025; visual cylinder length=0.05 radius=0.025
- link front_right_wheel: geometry collision cylinder length=0.05 radius=0.025; visual cylinder length=0.05 radius=0.025
- link rear_left_wheel: geometry collision cylinder length=0.05 radius=0.025; visual cylinder length=0.05 radius=0.025
- link rear_right_wheel: geometry collision cylinder length=0.05 radius=0.025; visual cylinder length=0.05 radius=0.025
Joints:
- joint front_left_wheel_joint: origin xyz=0.25 0.29 0.0 rpy=0 0 0 -> xyz=0.245 0.245 0.0 rpy=0 0 0
- joint front_right_wheel_joint: origin xyz=0.25 -0.29 0.0 rpy=0 0 0 -> xyz=0.245 -0.245 0.0 rpy=0 0 0
- joint rear_left_wheel_joint: origin xyz=-0.25 0.29 0.0 rpy=0 0 0 -> xyz=-0.245 0.245 0.0 rpy=0 0 0
- joint rear_right_wheel_joint: origin xyz=-0.25 -0.29 0.0 rpy=0 0 0 -> xyz=-0.245 -0.245 0.0 rpy=0 0 0

Commit message: stage

File: map/scout_mini_omni.urdf (robot description, URDF)
Before this commit: robot scout_mini_omni, 5 links, 4 joints
Links:
- link base_link: geometry collision box size=0.153 0.145 0.06125; visual box size=0.153 0.145 0.06125

Commit message: param

File: map/scout_mini_omni.urdf (robot description, URDF)
Before this commit: robot scout_mini_omni, 5 links, 4 joints
Links:
- removed link front_left_wheel
- removed link front_right_wheel
- removed link rear_left_wheel
- removed link rear_right_wheel
- link base_link: geometry collision box size=0.153 0.145 0.06125; visual box size=0.627 0.550 0.1
Joints:
- removed joint front_left_wheel_joint
- removed joint front_right_wheel_joint
- removed joint rear_left_wheel_joint
- removed joint rear_right_wheel_joint

Commit message: param

File: map/scout_mini_omni.urdf (robot description, URDF)
Before this commit: robot scout_mini_omni, 1 links, 0 joints
Links:
- link base_link: geometry collision box size=0.153 0.145 0.06125; visual box size=0.31 0.28 0.1
